File: KiCad/Master_sheet/LV_tiger_master_sheet.kicad_pcb (KiCad board)
At the start: 2 copper layers, 49 parts, among them J1 MSD-1-A, M1 NTR2101P, M2 NTR2101P, M3 NTR2101P, U1 ESP32-S3-DEVKITC-1-N8R8, U2 SN65HVD230, U3 TPS74801AWDRC, U4 LMR51430

Commit message: made some changes to pcb layout
Routing:
- net GND: track 50.5 -> 47.2 mm
Changed lines of the file:
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@@
 			(at 4.12 5.365 90)
 			(layer "F.Fab")
+			(hide yes)
 			(effects
 				(font
@@
 		(start 122.75 68.75)
 		(end 123.25 68.75)
-		(width 0.4)
-		(layer "F.Cu")
-		(net 2)
-	)
-	(segment
-		(start 167.29 67.75)
-		(end 168.895 67.75)
-		(width 0.4)
+		(width 0.6)
+		(layer "F.Cu")
+		(net 2)
+	)
+	(segment
+		(start 166.182 62.25)
+		(end 167 62.25)
+		(width 0.6)
 		(layer "F.Cu")
 		(net 2)
@@
 		(end 175.25 115.969)
 		(width 0.2)
+		(layer "F.Cu")
+		(net 2)
+	)
+	(segment
+		(start 142.815 61.885)
+		(end 141.5 61.885)
+		(width 0.6)
 		(layer "F.Cu")
 		(net 2)
@@
 	)
 	(segment
-		(start 167.29 64.75)
-		(end 168.895 64.75)
-		(width 0.4)
-		(layer "F.Cu")
-		(net 2)
-	)
-	(segment
-		(start 144.25 71.73)
-		(end 143.25 71.73)
-		(width 0.4)
+		(start 167.29 67.75)
+		(end 168.5 67.75)
+		(width 0.6)
 		(layer "F.Cu")
 		(net 2)
@@
 	)
 	(segment
-		(start 161.65 73.114)
-		(end 161.65 74.182)
-		(width 0.4)
-		(layer "F.Cu")
-		(net 2)
-	)
-	(segment
 		(start 148.5 66)
 		(end 148.25 66.25)
@@
 		(start 133.8 114.55)
 		(end 133.25 114)
-		(width 0.4)
+		(width 0.6)
 		(layer "F.Cu")
 		(net 2)
@@
 	)
 	(segment
-		(start 161.65 74.182)
-		(end 161.65 73.682)
-		(width 0.2)
-		(layer "F.Cu")
-		(net 2)
-	)
-	(segment
 		(start 149.8 66.5)
 		(end 149.34 66.5)
@@
 		(start 127.8 114.55)
 		(end 127.25 114)
-		(width 0.4)
+		(width 0.6)
 		(layer "F.Cu")
 		(net 2)
@@
 	)
 	(segment
-		(start 118.2 62)
-		(end 119.75 62)
-		(width 0.4)
-		(layer "F.Cu")
-		(net 2)
-	)
-	(segment
 		(start 148 66)
 		(end 148.25 66.25)
@@
 	)
 	(segment
-		(start 142.815 61.885)
-		(end 141.275 61.885)
-		(width 0.4)
-		(layer "F.Cu")
-		(net 2)
-	)
-	(segment
 		(start 175.75 121.305)
 		(end 175.75 122.75)
@@
 	)
 	(segment
-		(start 145.318 69.125)
-		(end 144.25 69.125)
-		(width 0.4)
-		(layer "F.Cu")
-		(net 2)
-	)
-	(segment
 		(start 176.385 104.275)
 		(end 176.385 102.01)
@@
 		(start 155.73 71.15)
 		(end 155.73 72.13)
-		(width 0.4)
+		(width 0.6)
 		(layer "F.Cu")
 		(net 2)
@@
 	)
 	(segment
+		(start 119.5 66.5)
+		(end 121 66.5)
+		(width 0.6)
+		(layer "F.Cu")
+		(net 2)
+	)
+	(segment
 		(start 139.8 116.295)
 		(end 139.8 114.55)
-		(width 0.4)
+		(width 0.6)
 		(layer "F.Cu")
 		(net 2)
@@
 		(start 139.25 112.48875)
 		(end 139.25 114)
-		(width 0.4)
+		(width 0.6)
 		(layer "F.Cu")
 		(net 2)
@@
 		(start 118.45 76.6)
 		(end 119.75 76.6)
-		(width 0.4)
-		(layer "F.Cu")
-		(net 2)
-	)
-	(segment
-		(start 108.9 62)
-		(end 108.9 60.4)
-		(width 0.4)
-		(layer "F.Cu")
-		(net 2)
-	)
-	(segment
-		(start 119.5 66.5)
-		(end 121 66.5)
-		(width 0.4)
+		(width 0.6)
+		(layer "F.Cu")
+		(net 2)
+	)
+	(segment
+		(start 161.65 73.114)
+		(end 161.65 74)
+		(width 0.6)
 		(layer "F.Cu")
 		(net 2)
@@
 		(start 127.25 112.48875)
 		(end 127.25 114)
-		(width 0.4)
+		(width 0.6)
 		(layer "F.Cu")
 		(net 2)
@@
 		(start 133.8 116.31625)
 		(end 133.8 114.55)
-		(width 0.4)
+		(width 0.6)
 		(layer "F.Cu")
 		(net 2)
@@
 		(start 133.25 112.5)
 		(end 133.25 114)
-		(width 0.4)
+		(width 0.6)
 		(layer "F.Cu")
 		(net 2)
@@
 	)
 	(segment
+		(start 167.29 64.75)
+		(end 168.5 64.75)
+		(width 0.6)
+		(layer "F.Cu")
+		(net 2)
+	)
+	(segment
 		(start 158.75 71.15)
 		(end 158.75 72.15)
-		(width 0.4)
+		(width 0.6)
 		(layer "F.Cu")
 		(net 2)
@@
 	)
 	(segment
-		(start 166.216 62.25)
-		(end 167.284 62.25)
-		(width 0.4)
-		(layer "F.Cu")
-		(net 2)
-	)
-	(segment
 		(start 127.8 116.31625)
 		(end 127.8 114.55)
-		(width 0.4)
+		(width 0.6)
+		(layer "F.Cu")
+		(net 2)
+	)
+	(segment
+		(start 118.2 62)
+		(end 119.5 62)
+		(width 0.6)
 		(layer "F.Cu")
 		(net 2)
@@
 		(start 139.8 114.55)
 		(end 139.25 114)
-		(width 0.4)
+		(width 0.6)
+		(layer "F.Cu")
+		(net 2)
+	)
+	(segment
+		(start 108.9 62)
+		(end 108.9 61)
+		(width 0.6)
 		(layer "F.Cu")
 		(net 2)
@@
 		(start 108.9 77.5)
 		(end 108.9 78.6)
-		(width 0.4)
+		(width 0.6)
 		(layer "F.Cu")
 		(net 2)
@@
 		(start 161.5125 61.3)
 		(end 160.2 61.3)
-		(width 0.4)
+		(width 0.6)
+		(layer "F.Cu")
+		(net 2)
+	)
+	(segment
+		(start 145.318 69.125)
+		(end 144.5 69.125)
+		(width 0.6)
 		(layer "F.Cu")
 		(net 2)
@@
 	)
 	(segment
+		(start 143.5 71.73)
+		(end 144.25 71.73)
+		(width 0.5)
+		(layer "F.Cu")
+		(net 2)
+	)
+	(segment
 		(start 122.182 68.75)
 		(end 122.75 68.75)
-		(width 0.4)
+		(width 0.6)
 		(layer "F.Cu")
 		(net 2)
@@
 	)
 	(via
-		(at 168.895 67.75)
-		(size 0.6)
-		(drill 0.3)
-		(layers "F.Cu" "B.Cu")
-		(net 2)
-	)
-	(via
-		(at 167.284 62.25)
+		(at 168.5 67.75)
+		(size 0.6)
+		(drill 0.3)
+		(layers "F.Cu" "B.Cu")
+		(net 2)
+	)
+	(via
+		(at 167 62.25)
 		(size 0.6)
 		(drill 0.3)
@@
 	)
 	(via
-		(at 119.75 62)
+		(at 119.5 62)
 		(size 0.6)
 		(drill 0.3)
@@
 	)
 	(via
-		(at 143.25 71.73)
+		(at 143.5 71.73)
 		(size 0.6)
 		(drill 0.3)
@@
 	)
 	(via
-		(at 141.275 61.885)
+		(at 141.5 61.885)
 		(size 0.6)
 		(drill 0.3)
@@
 	)
 	(via
-		(at 108.9 60.4)
-		(size 0.6)
-		(drill 0.3)
-		(layers "F.Cu" "B.Cu")
-		(net 2)
-	)
-	(via
-		(at 168.895 64.75)
+		(at 108.9 61)
+		(size 0.6)
+		(drill 0.3)
+		(layers "F.Cu" "B.Cu")
+		(net 2)
+	)
+	(via
+		(at 168.5 64.75)
 		(size 0.6)
 		(drill 0.3)
@@
 	)
 	(via
-		(at 161.65 74.182)
+		(at 161.65 74)
 		(size 0.6)
 		(drill 0.3)
@@
 	)
 	(via
-		(at 144.25 69.125)
-		(size 0.6)
-		(drill 0.3)
+		(at 144.5 69.125)
+		(size 0.6)
+		(drill 0.3)

Commit message: made a lot of revisions to the schematic, not yet updated pcb layout
Parts:
- removed CAN_signal_input1, Display_MCU1, Power_input1: Screw_Terminal_01x02, 691137710002:691137710002
- removed M1, M2, M3: NTR2101P, Package_TO_SOT_SMD:SOT-23
- removed Relay_control1: Screw_Terminal_01x03, 691214110003:691214110003
- added J2: Connector IN, DT13-12PA:DT13-12, F.Cu at (18.0, 57.3)
- added J3: Connector OUT, DT13-12PA:DT13-12, F.Cu at (60.6, 57.3)
- added K1: Precharge switch, Relay_THT:Relay_SPDT_Omron-G5Q-1, F.Cu at (101.1, 25.1)
- added K2: BMS switch, Relay_THT:Relay_SPDT_Omron-G5Q-1, F.Cu at (101.1, 37.6)
- added K3: HV switch, Relay_THT:Relay_SPDT_Omron-G5Q-1, F.Cu at (101.1, 50.2)
- added K4: Cooling switch, Relay_THT:Relay_SPDT_Omron-G5Q-1, F.Cu at (101.1, 62.8)
- added Q1: NTJS3151PT2G, KiCad:SOT65P210X110-6N, F.Cu at (105.7, 67.0)
- added Q2: NTJS3151PT2G, KiCad:SOT65P210X110-6N, F.Cu at (105.7, 70.6)
- added Q3: 2N7002K, Package_TO_SOT_SMD:SOT-23, F.Cu at (101.1, 67.6)
- added Q4: 2N7002K, Package_TO_SOT_SMD:SOT-23, F.Cu at (101.1, 72.2)
- added Q5: 2N7002K, Package_TO_SOT_SMD:SOT-23, F.Cu at (101.1, 76.9)
- added Q6: 2N7002K, Package_TO_SOT_SMD:SOT-23, F.Cu at (101.1, 81.5)
- added Q7: NTJS3151PT2G, KiCad:SOT65P210X110-6N, F.Cu at (105.7, 74.2)
- added Q8: NTJS3151PT2G, KiCad:SOT65P210X110-6N, F.Cu at (105.7, 77.8)
- added R15: 10kΩ, RC0603FR-0710KL:RESC1607X60N, F.Cu at (100.3, 126.5)
- added R16: 100 kΩ, RC0402FR-07100KL:RESC1005X40, F.Cu at (96.6, 123.6)
- added R17: 100 kΩ, RC0402FR-07100KL:RESC1005X40, F.Cu at (109.7, 66.4)
- added R18: 100 kΩ, RC0402FR-07100KL:RESC1005X40, F.Cu at (109.7, 68.7)
- added R19: 100 kΩ, RC0402FR-07100KL:RESC1005X40, F.Cu at (109.7, 71.0)
- added R20: 1.6kΩ, RC1206JR-071K6L:RESC3116X65N, F.Cu at (114.1, 66.9)
- added R21: 10kΩ, RC0603FR-0710KL:RESC1607X60N, F.Cu at (142.0, 78.0)
- moved LOGO_placeholder1 92.5 mm to (41.0, 177.5)
- moved R14 22.6 mm to (142.0, 76.0)
- moved C4 21.5 mm to (194.4, 127.8)
- moved C5 21.5 mm to (193.0, 127.8)
- moved R4 21.5 mm to (145.2, 123.6)
- moved R6 21.5 mm to (157.2, 123.6)
- moved R7 21.5 mm to (147.8, 124.1)
- moved R8 21.5 mm to (153.8, 124.1)
- moved CIN3 21.5 mm to (162.3, 73.7)
- moved C1 21.5 mm to (193.8, 111.6)
- moved C2 21.5 mm to (193.8, 113.6)
- moved C3 21.5 mm to (193.8, 125.6)
- moved C6 21.5 mm to (139.8, 80.6)
- moved CBOOT1 21.5 mm to (180.7, 71.1)
- moved CFF1 21.5 mm to (164.8, 85.9)
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Connections:
- net /12V in renamed +12V
- R4 pad 2: GND -> +3V3
- R5 pad 2: GND -> +3V3
- R6 pad 2: GND -> +3V3
- U1 pad J3_10: unconnected-(U1-GPIO38-PadJ3_10) -> /GPIO 38
Routing:
- net /GPIO18 (RX): track 22.1 -> 0.00 mm
- net /GPIO17 (TX): track 22.0 -> 0.00 mm
- net GND: track 47.2 -> 35.0 mm, vias 24 -> 21
- net +3V3: track 100.5 -> 112.2 mm, vias 0 -> 3
- net /M3 drain: track 10.4 -> 0.00 mm
- net /M1 drain: track 10.3 -> 0.00 mm
- net /M2 drain: track 9.31 -> 0.00 mm
- net /MISO: track 20.7 -> 24.8 mm
- net Net-(J1-DAT1): track 2.54 -> 3.89 mm
- removed copper zone on B.Cu, net GND
