File: KiCad/Master_sheet/LV_tiger_master_sheet.kicad_sch (KiCad schematic)
At the start: 42 parts, among them M1 NTR2101P, M2 NTR2101P, M3 NTR2101P, U1 SN65HVD230, U2 TPS74801AWDRC, U3 LMR51430, U4 ESP32-S3-DEVKITC-1-N8R8

Commit message: finished PCB
Parts:
- removed C1: 4.7nF, Capacitor_SMD:CP_Elec_5x3, symbol Device:C
- removed C2, C3: 30pF, Capacitor_SMD:CP_Elec_5x3, symbol Device:C
- removed C4: 0.1uF, Capacitor_SMD:CP_Elec_5x3, symbol Device:C
- removed C5: 4.7uF, Capacitor_SMD:CP_Elec_5x3, symbol Device:C
- removed CFF1: 10 nF, symbol Device:C
- removed CIN1, CIN2: 4.7uF, symbol Device:C_Small
- removed CIN1: 0.1uF, symbol Device:C_Small
- removed CIN3: 10 µF, symbol Device:C
- removed CNR/SS1: 10 nF to 1 µF, symbol Device:C
- removed COUT1: 47 µF, symbol Device:C
- removed C_BOOT1: 0.1 µF, symbol Device:C_Small
- removed C_OUT1, C_OUT2: 22 µF, symbol Device:C_Small
- added C1, C6, CBOOT1, CIN5: 0.1uF, CL05A104KA5NNNC:CAPC1005X55N, symbol CL05A104KA5NNNC:CL05A104KA5NNNC
- added C2, CIN2, CIN4: 4.7uF, CL21A475KAQNNNE:CAPC2012X140N, symbol CL21A475KAQNNNE:CL21A475KAQNNNE
- added C3: 4.7nF, CL05A104KA5NNNC:CAPC1005X55N, symbol CL10A475KP8NNNC:CL10A475KP8NNNC
- added C4, C5: 30pF, GRM0335C1E300JA01D:CAPC0603X33N, symbol GRM0335C1E300JA01D:GRM0335C1E300JA01D
- added CFF1, CNR/SS1: 10nF, CL05B103KO5NNNC:CAPC1005X55N, symbol CL05B103KO5NNNC:CL05B103KO5NNNC
- added CIN1: 10uF, WCAP-ATG5_5X11:WCAP-ATG5_5X11_DXL_, symbol WCAP-ATG5_5X11:WCAP-ATG5_5X11
- added CIN3: 10uF, CL31B106KAHNNNE:CAPC3216X180N, symbol CL31B106KAHNNNE:CL31B106KAHNNNE
- added COUT1: 47uF, CL21A476MQYNNNG:CAPC2012X145N, symbol CL21A476MQYNNNG:CL21A476MQYNNNG
- added COUT2, COUT3: 22uF, CL21A226MAYNNNE:CAPC2012X145N, symbol CL21A226MAYNNNE:CL21A226MAYNNNE
- added J1: MSD-1-A, MSD-1-A:CUI_MSD-1-A, symbol MSD-1-A:MSD-1-A
- added LOGO_placeholder1: C, pes_logo:new_pes_logo, symbol Device:C
- added R12, R13, R14: 10kΩ, RC0603FR-0710KL:RESC1607X60N, symbol Device:R_US
- CAN_signal_input1, Display_MCU1, Power_input1: footprint (none) -> 691137710002:691137710002
- L1: footprint (none) -> VLS6045EX-6R8M:IND_VLS6045EX-6R8M
- R1: renamed from R3; footprint Resistor_SMD:R_0201_0603Metric_Pad0.64x0.40mm_HandSolder -> RMCF0603FT1K00:RESC1508X55N
- R10: renamed from R4; footprint (none) -> RC0402FR-1311K8L:RESC1005X40N
- R11: renamed from R5; footprint (none) -> RC0201FR-073K74L:RESC0603X26N
- R4: renamed from R7; footprint (none) -> RC0603FR-0710KL:RESC1607X60N
- R5: renamed from R8; footprint (none) -> RC0603FR-0710KL:RESC1607X60N
- R6: renamed from R10; footprint (none) -> RC0603FR-0710KL:RESC1607X60N
- R7: renamed from R6; footprint (none) -> RC1206JR-071K6L:RESC3116X65N
- R8: renamed from R9; footprint (none) -> RC1206JR-071K6L:RESC3116X65N
- R9: renamed from R11; footprint (none) -> RC1206JR-071K6L:RESC3116X65N
- RPG1: value 10 kΩ - 100 kΩ -> 10 kΩ; footprint (none) -> RC0603FR-0710KL:RESC1607X60N
- R_FBB1: footprint (none) -> RC0402FR-0713K7L:RESC1005X40N
- R_FBT1: footprint (none) -> RC0402FR-07100KL:RESC1005X40
- Relay_control1: footprint (none) -> 691214110003:691214110003
- renumbered R1 to R2, R2 to R3, U4 to U1, U1 to U2, U2 to U3, U3 to U4
Connections:
- net Buck converter input is gone; now on net 12V in: Power_input1.1 (Pin_1)
- net CAN Transciver D pin is gone; now on net ESP RX pin: U1.J1_4 (GPIO4)
- net CAN Transciver R pin is gone; now on net ESP TX pin: U1.J1_5 (GPIO5)
- net CAN terminal block pin 1 is gone; now on net CAN H: D1.1, R2.1, U2.7 (CANH)
- net CAN terminal block pin 2 is gone; now on net CAN L: D1.2, R3.2, U2.6 (CANL)
- net GNDREF is gone; now on net COVER_GND: R11.2, U3.11 (GND), U3.6 (GND)
- net M1 gate is gone; now on net GPIO 35: U1.J3_13 (GPIO35)
- net M2 gate is gone; now on net GPIO 36: U1.J3_12 (GPIO36)
- net M3 gate is gone; now on net GPIO 37: U1.J3_11 (GPIO37)
- net Pin 1 of Relay terminal block is gone; now on net M1 drain: M1.3 (D)
- net Pin 2 of Relay terminal block is gone; now on net M2 drain: M2.3 (D)
- net Pin 3 of Relay terminal block is gone; now on net M3 drain: M3.3 (D)
- net To Load is gone; now on net +3V3: R10.1, RPG1.2, U3.9 (OUT)
- net Vin for LDO is gone; now on net Vin LDO: L1.2, R_FBT1.1
- net +3V3: now also C1.1, C2.1, C6.1, CFF1.1, COUT1.1, J1.4 (VDD), R12.1, R13.1, R14.1
- net CAN H: now also CAN_signal_input1.2 (Pin_2), C4.1; no longer CAN_signal_input1.1 (Pin_1)
- net CAN L: now also CAN_signal_input1.1 (Pin_1), C5.1; no longer CAN_signal_input1.2 (Pin_2)
- net GPIO17 (TX): now also Display_MCU1.2 (Pin_2), U1.J3_2 (U0TXD/GPIO43); no longer Display_MCU1.1 (Pin_1)
- net GPIO18 (RX): now also Display_MCU1.1 (Pin_1), U1.J3_3 (U0RXD/GPIO44); no longer Display_MCU1.2 (Pin_2)
- net at R10.2, R11.1, U3.8 (FB): now also CFF1.2, COUT1.2
- net at L1.1, U4.2 (SW): now also CBOOT1.2
- net at U4.6 (CB): now also CBOOT1.1
- net at R2.2, R3.1, U2.5 (Vref): now also C3.1
- net CS: now reaches U1.J1_16 (GPIO10)
- net CS: now also J1.2 (CD/DAT3), R12.2
- net MOSI: now reaches U1.J1_17 (GPIO11)
- net MOSI: now also J1.3 (CMD)
- net SCK: now reaches U1.J1_18 (GPIO12)
- net SCK: now also J1.5 (CLK)
- net MISO: now reaches U1.J1_19 (GPIO13)
- net MISO: now also J1.7 (DAT0)
- net at U3.7 (SS): now also CNR/SS1.1
- net 12V battery input (terminal blcok) renamed 12V in
- net 12V in: now also CIN1.1, CIN2.1, CIN4.1, CIN5.1
- net Display terminal block pin 1: no longer names the net of U1.J1_10 (GPIO17)
- net Display terminal block pin 2: no longer names the net of U1.J1_11 (GPIO18)
- net GND renamed COVER_GND
- net COVER_GND: now also C1.2, C2.2, C3.2, C4.2, C5.2, C6.2, CIN1.2, CIN2.2, CIN3.2, CIN4.2, CIN5.2, CNR/SS1.2, COUT2.2, COUT3.2, J1.6 (VSS), J1.G1 (COVER_GND), J1.G2 (COVER_GND), J1.G3 (COVER_GND), J1.G4 (COVER_GND)
- net Input Supply renamed Vin LDO
- net Vin LDO: now also CIN3.1, COUT2.1, COUT3.1
- new net: J1.1 (DAT2), R13.2
- new net: J1.8 (DAT1), R14.2
Other:
- moved on the sheet: RPG1

Commit message: made a lot of revisions to the schematic, not yet updated pcb layout
Parts:
- removed CAN_signal_input1, Display_MCU1, Power_input1: Screw_Terminal_01x02, 691137710002:691137710002, symbol Connector:Screw_Terminal_01x02
- removed M1, M2, M3: NTR2101P, Package_TO_SOT_SMD:SOT-23, symbol Transistor_FET:NTR2101P
- removed Relay_control1: Screw_Terminal_01x03, 691214110003:691214110003, symbol Connector:Screw_Terminal_01x03
- added F1, F2, F3, F4, F5, F6: ERB-RD0R50X, ERB-RD0R50X:FUSC0402X49N, symbol ERB-RD0R50X:ERB-RD0R50X
- added J2: Connector IN, DT13-12PA:DT13-12, symbol DT13-12PA:DT13-12PA
- added J3: Connector OUT, DT13-12PA:DT13-12, symbol DT13-12PA:DT13-12PA
- added K1: Precharge switch, Relay_THT:Relay_SPDT_Omron-G5Q-1, symbol Relay:G5Q-1
- added K2: BMS switch, Relay_THT:Relay_SPDT_Omron-G5Q-1, symbol Relay:G5Q-1
- added K3: HV switch, Relay_THT:Relay_SPDT_Omron-G5Q-1, symbol Relay:G5Q-1
- added K4: Cooling switch, Relay_THT:Relay_SPDT_Omron-G5Q-1, symbol Relay:G5Q-1
- added Q1, Q2, Q7, Q8: NTJS3151PT2G, KiCad:SOT65P210X110-6N, symbol NTJS3151PT2G:NTJS3151PT2G
- added Q3, Q4, Q5, Q6: 2N7002K, Package_TO_SOT_SMD:SOT-23, symbol Transistor_FET:2N7002K
- added R15, R21: 10kΩ, RC0603FR-0710KL:RESC1607X60N, symbol Device:R_US
- added R16, R17, R18, R19: 100 kΩ, RC0402FR-07100KL:RESC1005X40, symbol Device:R_US
- added R20: 1.6kΩ, RC1206JR-071K6L:RESC3116X65N, symbol Device:R_US
Connections:
- net +3V3: now also R4.2, R5.2, R6.2, Q3.2 (S), Q4.2 (S), Q5.2 (S), Q6.2 (S), R15.2, R21.1
- net CAN H: now also J3.2
- net CAN L: now also J3.1
- net COVER_GND: now also J2.12, J3.12, K1.1, K2.1, K3.1, K4.1; no longer R4.2, R5.2, R6.2
- net GPIO17 (TX): now also J2.7
- net GPIO18 (RX): now also J2.8
- net MISO: now also R21.2
- net at R9.1: now also Q5.1 (G)
- net at R8.1: now also Q4.1 (G)
- net GPIO 38: now reaches U1.J3_10 (GPIO38)
- net GPIO 38: now also R15.1, R20.2
- net at R7.1: now also Q3.1 (G)
- net 12V in renamed +12V
- net +12V: now also F1.1, Q1.4 (S), Q2.4 (S), Q7.4 (S), Q8.4 (S), R16.1, R17.1, R18.1, R19.1
- new net: Q1.3 (G), Q3.3 (D), R16.2
- new net: Q2.3 (G), Q4.3 (D), R17.2
- new net: F1.2, J2.1
- new net: F2.2, J2.2
- new net: F3.2, J2.3
- new net: F4.2, J2.4
- new net: F5.2, J2.5
- new net: F6.2, J2.6
- new net: Q5.3 (D), Q7.3 (G), R18.2
- new net: Q6.3 (D), Q8.3 (G), R19.2
- new net: Q6.1 (G), R20.1
- new net BMS: J3.4, K2.2
- new net BMS Relay: K2.4, Q2.1 (D_1), Q2.2 (D_2), Q2.5 (D_3), Q2.6 (D_4)
- new net Cooling: J3.6, K4.2
- new net Cooling Relay: K4.4, Q8.1 (D_1), Q8.2 (D_2), Q8.5 (D_3), Q8.6 (D_4)
- new net HV: J3.5, K3.2
- new net HV relay: K3.4, Q7.1 (D_1), Q7.2 (D_2), Q7.5 (D_3), Q7.6 (D_4)
- new net Override BMS: F4.1, K2.3
- new net Override Cooling: F5.1, K4.3
- new net Override HV: F3.1, K3.3
- new net Override Precharge: F2.1, K1.3
- new net Override Signal: F6.1, K1.5, K2.5, K3.5, K4.5
- new net Precharge: J3.3, K1.2
- new net Precharge Relay: K1.4, Q1.1 (D_1), Q1.2 (D_2), Q1.5 (D_3), Q1.6 (D_4)
Other:
- moved on the sheet: C1, C2, C3, C4, C5, C6, CBOOT1, CFF1, CIN1, CIN2, CIN3, CIN4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
